File: Narrow AAA sensor v1.sch (EAGLE design)
At the start: 16 parts, among them U1 ATMEGA328P_PDIP

Commit message: FIXed missing TMP wire
Connections:
- removed net A2: U1.PC2(ADC2)
- removed net A3: U1.PC3(ADC3)
- removed net B0: R4.1, TMP.DQ
- removed net D7: U1.PD7(AIN1)
- new net TMP: R4.1, TMP.DQ, U1.PB0(ICP)
