File: Narrow AAA sensor.sch (EAGLE design)
At the start: 16 parts, among them IC1 LD117AS33TR, U1 ATMEGA328P_PDIP

Commit message: https://PCBs.io/share/zM3DO
Parts:
- removed J2: (no value), SparkFun-Connectors:M02PTH
- added A0-GND: Analog, SparkFun-Connectors:M02PTH
- added D2: (no value), pinhead:PINHD-1X1
- added RA0: 10K, rcl:R-EU_0204/7
- SERIAL: device pinhead:PINHD-1X4 -> pinhead:PINHD-1X5
- VCC-D-GND-GND: value (none) -> Sensor
- renumbered R3 to R6, SENSOR to VCC-D-GND-GND
Connections:
- removed net A1: U1.PC1(ADC1)
- removed net D3: J2.2, U1.PD3(INT1)
- new net RESET: SERIAL.5, U1.PC6(/RESET)
- net A0: now also A0-GND.1, RA0.1
- net D2: now also D2.1; no longer J2.1
- net GND: now also A0-GND.2, SERIAL.2; no longer SERIAL.4
- net RXD: now also SERIAL.4; no longer SERIAL.2
- net VCC: now also RA0.2; no longer U1.PC6(/RESET)
Other:
- moved on the sheet: J3
